File: quad_robot_files/kicad_quad_1/quad_robot.kicad_pcb (KiCad board)
At the start: 2 copper layers, 99.1 x 95.8 mm, 25 parts, among them J1 Conn_01x02, J10 Conn_01x03, J11 Conn_01x03, J12 Conn_01x03, J13 Conn_01x03, J14 Conn_01x03, J15 Conn_01x04, J16 Conn_01x04, J2 Conn_01x03, J3 Conn_01x03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

Commit message: Add files via upload
Parts:
- added F1: Polyfuse_Small, Fuse:Fuse_BelFuse_0ZRE0055FF_L14.0mm_W4.1mm, F.Cu at (139.6, 107.6)
- SW1: value SW_SPDT -> SW_DPDT_x2
Connections:
- net Net-(J1-Pin_2) renamed +BATT
- C1 pad 1: Net-(D1-K) -> +VSW
- D1 pad 1: Net-(D1-K) -> +5VD
- J15 pad 2: +5V -> +5VD
- MD1 pad 2: Net-(D1-K) -> +VSW
- R1 pad 1: Net-(D1-K) -> +VSW
- SW1 pad 1: Net-(D1-A) -> Net-(SW1A-A)
- SW1 pad 4: (no net) -> unconnected-(SW1B-A-Pad4)
- SW1 pad 5: (no net) -> +5V
- SW1 pad 6: (no net) -> Net-(D1-A)
- U1 pad 39: +5V -> +5VD
Routing:
- net GND: track 570.6 -> 250.6 mm
- net Net-(SW1A-A): track 0.00 -> 45.9 mm
- net +5VD: track 0.00 -> 40.3 mm
- net +5V: track 113.9 -> 82.8 mm, vias 1 -> 0
- net +VSW: track 0.00 -> 29.3 mm
- net Net-(D1-K): track 24.3 -> 0.00 mm
- net Net-(D1-A): track 9.61 -> 6.31 mm
- added copper zone on B.Cu, net (none)
- added copper zone on F.Cu, net (none)
