File: quad_robot_files/kicad_quad_1/quad_robot.kicad_sch (KiCad schematic)
At the start: 25 parts, among them J1 Conn_01x02, J10 Conn_01x03, J11 Conn_01x03, J12 Conn_01x03, J13 Conn_01x03, J14 Conn_01x03, J15 Conn_01x04, J16 Conn_01x04, J2 Conn_01x03, J3 Conn_01x03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

Commit message: Add files via upload
Parts:
- removed SW1: SW_SPDT, Button_Switch_THT:SW_CK_JS202011CQN_DPDT_Straight, symbol Switch:SW_SPDT
- added F1: Polyfuse_Small, Fuse:Fuse_BelFuse_0ZRE0055FF_L14.0mm_W4.1mm, symbol Device:Polyfuse_Small
- added SW1: SW_DPDT_x2, Button_Switch_THT:SW_CK_JS202011CQN_DPDT_Straight, symbol Switch:SW_DPDT_x2
Connections:
- net +5V: now also SW1.5 (B); no longer J15.2 (Pin_2), U1.39 (VSYS)
- net +VSW: now reaches C1.1, MD1.2 (VIN), R1.1
- net +VSW: now also F1.2; no longer D1.1 (K)
- net at D1.2 (A): now also SW1.6 (C)
- net +BATT: now reaches J1.2 (Pin_2)
- net +BATT: now also SW1.2 (B)
- new net: F1.1, SW1.1 (A)
- new net +5VD: D1.1 (K), J15.2 (Pin_2), U1.39 (VSYS)
- no-connect marks 24 -> 25
Other:
- moved on the sheet: C1, C2, D1, J1, J10, J11, J12, J13, J14, J15, J16, J2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
